Commit message: first_commit

File: sampling_based_control/mppi_examples/mppi_manipulation/data/panda_mobile.urdf.xacro (robot description, xacro)
@@ -8,4 +8,11 @@
     <link name="world"/>
     <!--    Omnidirectional base-->
+    <!-- <xacro:unless value="$(arg fixed_base)">
+        <joint name="world_joint" type="fixed">
+            <parent link="world"/>
+            <child link="omni_base_root_link"/>
+        </joint>
+        <xacro:planar_base connect_to="base_link"/>
+    </xacro:unless> -->
     <xacro:unless value="$(arg fixed_base)">
         <joint name="world_joint" type="fixed">
@@ -15,4 +22,11 @@
         <xacro:planar_base connect_to="base_link"/>
     </xacro:unless>
+    <!-- <xacro:if value="$(arg fixed_base)">
+        <joint name="world_joint" type="fixed">
+            <parent link="world"/>
+            <child link="base_link"/>
+             <origin xyz="-0.5265965085817698 -0.2806388380571893 0.0" rpy="0.000 0.000 -0.04332860681335808"/>
+        </joint>
+    </xacro:if> -->
     <xacro:if value="$(arg fixed_base)">
         <joint name="world_joint" type="fixed">
@@ -23,10 +37,18 @@
     </xacro:if>
     <!--   Ridgeback base: for collision and appearance -->
-    <xacro:ridgeback/>
+    <!-- <xacro:ridgeback/> -->
+    <xacro:include filename="$(find fr3_xls_moveit_config)/config/summit_xl.urdf"/>
     <!--Mount panda on ridgeback-->
+    <!-- <joint name="arm_mount_joint" type="fixed"> -->
+        <!-- <parent link="mid_mount"/> -->
+        <!-- <child link="franka_mount_link"/> -->
+        <!--        <origin xyz="$(optenv RIDGEBACK_FRANKA_XYZ 0.21 0.0 0.2)" rpy="$(optenv RIDGEBACK_FRANKA_RPY 0 0 0)"/>-->
+        <!-- <origin xyz="0.295 0.005 0.445" rpy="0 0 0"/> -->
+    <!-- </joint> -->
+    <!-- <link name="franka_mount_link"/> -->
+    <!-- <xacro:panda_robot parent_link="franka_mount_link"/> -->
     <joint name="arm_mount_joint" type="fixed">
-        <parent link="mid_mount"/>
+        <parent link="base_link"/>
         <child link="franka_mount_link"/>
-        <!--        <origin xyz="$(optenv RIDGEBACK_FRANKA_XYZ 0.21 0.0 0.2)" rpy="$(optenv RIDGEBACK_FRANKA_RPY 0 0 0)"/>-->
         <origin xyz="0.295 0.005 0.445" rpy="0 0 0"/>
     </joint>

File: sampling_based_control/mppi_examples/mppi_manipulation/data/panda_mobile_gazebo.urdf.xacro (robot description, xacro)
@@ -3,10 +3,18 @@
     <xacro:include filename="$(find mppi_panda)/resources/panda/panda.urdf.xacro"/>
     <xacro:include filename="$(find mppi_manipulation)/data/planar_base.urdf.xacro"/>
-    <xacro:include filename="$(find mppi_manipulation)/data/ridgeback.urdf.xacro"/>
+    <!-- <xacro:include filename="$(find mppi_manipulation)/data/ridgeback.urdf.xacro"/>
     <xacro:ridgeback/>
-    <xacro:include filename="$(find mppi_manipulation)/data/ridgeback_gazebo.urdf.xacro"/>
+    <xacro:include filename="$(find mppi_manipulation)/data/ridgeback_gazebo.urdf.xacro"/> -->
+    <xacro:include filename="$(find fr3_xls_moveit_config)/config/gazebo_summit_xl.urdf"/>
     <!--Mount panda on ridgeback-->
+    <!-- <joint name="arm_mount_joint" type="fixed">
+        <parent link="mid_mount"/>
+        <child link="franka_mount_link"/>
+        <origin xyz="0.30 0.0 0.445" rpy="0 0 0"/>
+    </joint>
+    <link name="franka_mount_link"/>
+    <xacro:panda_robot parent_link="franka_mount_link" robot_description="/robot_description_for_gazebo"/> -->
     <joint name="arm_mount_joint" type="fixed">
-        <parent link="mid_mount"/>
+        <parent link="base_link"/>
         <child link="franka_mount_link"/>
         <origin xyz="0.30 0.0 0.445" rpy="0 0 0"/>

File: sampling_based_control/mppi_examples/mppi_panda/resources/panda/panda.urdf.xacro (robot description, xacro)
@@ -8,5 +8,5 @@
     <xacro:arg name="collision_finger" default="true"/>
     <xacro:arg name="custom_fingers" default="false"/>
-    <xacro:arg name="no_position_limits" default="true"/>
+    <xacro:arg name="no_position_limits" default="false"/>
     <xacro:arg name="friction" default="0.0"/>
     <xacro:arg name="damping"  default="0.0"/>
