Commit message: Applied DBB method for self-collision avoidance

File: fr3_xls_moveit_config/config/gazebo_summit_xl.urdf (robot description, URDF)
Before this commit: robot summit_xl, 29 links, 28 joints
Links:
- added link dbb_collision_link; visual mesh filename=package://mppi_royalpanda/mesh/DBB_mesh.obj
Joints:
- added joint dbb_collision_joint: type fixed, parent base_link, child dbb_collision_link, origin xyz=0.0 0 0.0 rpy=0 0 0

File: sampling_based_control/mppi_examples/mppi_panda/resources/panda/panda.urdf.xacro (robot description, xacro)
@@ -311,5 +311,5 @@
         </link>
         <joint name="panda_joint_4_1" type="fixed">
-            <origin rpy="0 0 0" xyz="-0.08 0 0"/>
+            <origin rpy="0 0 0" xyz="-0.0825 0 0"/>
             <parent link="panda_link4"/>
             <child link="panda_link_4_1"/>
