Commit message: Added self collision cost

File: sampling_based_control/mppi_examples/mppi_panda/resources/panda/panda.urdf.xacro (robot description, xacro)
@@ -40,4 +40,5 @@
         <gazebo reference="panda_link3"/>
         <gazebo reference="panda_link4"/>
+        <gazebo reference="panda_link_intermediate"/>
         <gazebo reference="panda_link5"/>
         <gazebo reference="panda_link6"/>
@@ -293,4 +294,18 @@
             </xacro:unless>
             <dynamics damping="${damping}" friction="${friction}"/>
+        </joint>
+        <link name="panda_link_4_1">
+            <inertial>
+                <mass value="0.01"/>
+                <origin rpy="0 0 0" xyz="0 0 0"/>
+                <inertia ixx="0.00799663881132" ixy="0.00347095570217" ixz="-0.00241222942995" iyy="0.00825390705278"
+                         iyz="0.00235774044121" izz="0.0102515004345"/>
+            </inertial>
+        </link>
+        <joint name="panda_joint_4_1" type="fixed">
+            <origin rpy="0 0 0" xyz="-0.08 0 0"/>
+            <parent link="panda_link4"/>
+            <child link="panda_link_4_1"/>
+            <axis xyz="0 0 1"/>
         </joint>
         <link name="panda_link5">

Commit message: Added DBB self-collision-avidance and input filter

File: sampling_based_control/mppi_examples/mppi_panda/resources/panda/panda.urdf.xacro (robot description, xacro)
@@ -40,4 +40,5 @@
         <gazebo reference="fr3_link3"/>
         <gazebo reference="fr3_link4"/>
+        <gazebo reference="fr3_link_4_1"/>
         <gazebo reference="fr3_link5"/>
         <gazebo reference="fr3_link6"/>
@@ -293,4 +294,18 @@
             </xacro:unless>
             <dynamics damping="${damping}" friction="${friction}"/>
+        </joint>
+        <link name="fr3_link_4_1">
+            <inertial>
+                <mass value="0.01"/>
+                <origin rpy="0 0 0" xyz="0 0 0"/>
+                <inertia ixx="0.00799663881132" ixy="0.00347095570217" ixz="-0.00241222942995" iyy="0.00825390705278"
+                         iyz="0.00235774044121" izz="0.0102515004345"/>
+            </inertial>
+        </link>
+        <joint name="fr3_joint_4_1" type="fixed">
+            <origin rpy="0 0 0" xyz="-0.0825 0 0"/>
+            <parent link="fr3_link4"/>
+            <child link="fr3_link_4_1"/>
+            <axis xyz="0 0 1"/>
         </joint>
         <link name="fr3_link5">
